Commit message: feat(indicator): add advanced light patterns for safety states
- Added Blinking Red (0.5s) for Super Override
- Added Solid Dark Yellow for Obstacle Safety Stop
- Added Blinking Cyan for Localization Invalid
- Added Blinking Yellow for Manual Override
- Implemented state prioritization and dynamic blink frequencies

File: src/next2_motor/description/robot.urdf.xacro (robot description, xacro)
@@ -11,4 +11,5 @@
     </xacro:unless> -->
     <xacro:include filename="lidar.xacro" />
+    <!-- <xacro:include filename="imu2.xacro" /> -->
     <!-- <xacro:include filename="camera.xacro" /> -->
     <!-- <xacro:include filename="depth_camera.xacro" /> -->

File: src/next2_motor/description/robot_core.xacro (robot description, xacro)
@@ -253,16 +253,16 @@
         <parent link="chassis"/>
         <child link="imu_link"/>
-        <origin xyz="0.40 0 0.055" rpy="0 0 0"/>
+        <origin xyz="0.4 0 0.10" rpy="0 0 0"/>
     </joint>
     <link name="imu_link">
         <visual>
             <geometry>
-                <box size="0.05 0.05 0.05"/>
-            </geometry>
-            <material name="red"/>
-        </visual>
-        <collision>
-            <geometry>
-                <box size="0.05 0.05 0.05"/>
+                <box size="0.0538 0.0488 0.0252"/>
+            </geometry>
+            <material name="red"/>
+        </visual>
+        <collision>
+            <geometry>
+                <box size="0.0538 0.0488 0.0252"/>
             </geometry>
         </collision>
